File: power_stage.kicad_sch (KiCad schematic)
At the start: 25 parts, among them U1 OPA567AIRHGR, U2 INA199A1DCKR

Commit message: More layout
Parts:
- added C3: 0.1u, passive:C_0402, symbol Device:C_Small
- added R1 (x2): 100k, passive:R_0402, symbol Device:R_Small
Connections:
- net GND: now also C3.2, R1.1
- net V_{O}: now also R1.2
- new net V_{MEAS}: C3.1, R1.1, R1.2
Changed lines of the file:
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@@
   (junction (at 201.93 90.17) (diameter 0) (color 0 0 0 0)
   )
+  (junction (at 130.81 139.7) (diameter 0) (color 0 0 0 0)
+  )
   (junction (at 168.91 90.17) (diameter 0) (color 0 0 0 0)
   )
@@
     (stroke (width 0) (type default))
   )
+  (wire (pts (xy 130.81 137.16) (xy 130.81 139.7))
+    (stroke (width 0) (type default))
+  )
   (wire (pts (xy 168.91 90.17) (xy 168.91 93.98))
     (stroke (width 0) (type default))
@@
     (stroke (width 0) (type default))
   )
+  (wire (pts (xy 130.81 129.54) (xy 130.81 132.08))
+    (stroke (width 0) (type default))
+  )
+  (wire (pts (xy 140.97 139.7) (xy 140.97 142.24))
+    (stroke (width 0) (type default))
+  )
   (wire (pts (xy 212.09 90.17) (xy 222.25 90.17))
     (stroke (width 0) (type default))
@@
     (stroke (width 0) (type default))
   )
+  (wire (pts (xy 130.81 139.7) (xy 140.97 139.7))
+    (stroke (width 0) (type default))
+  )
+  (wire (pts (xy 123.19 139.7) (xy 130.81 139.7))
+    (stroke (width 0) (type default))
+  )
   (wire (pts (xy 222.25 90.17) (xy 229.87 90.17))
     (stroke (width 0) (type default))
@@
   )
   (wire (pts (xy 116.84 90.17) (xy 116.84 78.74))
+    (stroke (width 0) (type default))
+  )
+  (wire (pts (xy 130.81 139.7) (xy 130.81 142.24))
     (stroke (width 0) (type default))
   )
@@
     (effects (font (size 1.27 1.27)) (justify right bottom))
   )
+  (label "V_{O}" (at 130.81 129.54 180) (fields_autoplaced)
+    (effects (font (size 1.27 1.27)) (justify right bottom))
+  )
   (hierarchical_label "VREF_PWM" (shape input) (at 44.45 86.36 180) (fields_autoplaced)
     (effects (font (size 1.27 1.27)) (justify right))
@@
     (effects (font (size 1.27 1.27)) (justify left))
   )
+  (hierarchical_label "V_{MEAS}" (shape input) (at 123.19 139.7 180) (fields_autoplaced)
+    (effects (font (size 1.27 1.27)) (justify right))
+  )
   (hierarchical_label "OVERTEMP" (shape input) (at 120.65 102.87 0) (fields_autoplaced)
     (effects (font (size 1.27 1.27)) (justify left))
@@
         (path "/7161d457-3f04-48e1-b7cc-1aacc3ce662e/5cf08dfe-d906-4adb-8c99-60cc69db1b65"
           (reference "R13") (unit 1)
+        )
+      )
+    )
+  )
+  (symbol (lib_id "Device:R_Small") (at 130.81 134.62 180) (unit 1)
+    (in_bom yes) (on_board yes) (dnp no) (fields_autoplaced)
+    (property "Reference" "R1" (at 133.35 133.35 0)
+      (effects (font (size 1.27 1.27)) (justify right))
+    )
+    (property "Value" "100k" (at 133.35 135.89 0)
+      (effects (font (size 1.27 1.27)) (justify right))
+    )
+    (property "Footprint" "passive:R_0402" (at 130.81 134.62 0)
+      (effects (font (size 1.27 1.27)) hide)
+    )
+    (property "Datasheet" "~" (at 130.81 134.62 0)
+      (effects (font (size 1.27 1.27)) hide)
+    )
+    (property "MFPN" "" (at 130.81 134.62 0)
+      (effects (font (size 1.27 1.27)) hide)
+    )
+    (property "Specification" "" (at 130.81 134.62 0)
+      (effects (font (size 1.27 1.27)) hide)
+    )
+    (pin "1")
+    (pin "2")
+    (instances
+      (project "battery-emulator"
+        (path "/7161d457-3f04-48e1-b7cc-1aacc3ce662e"
+          (reference "R1") (unit 1)
+        )
+        (path "/7161d457-3f04-48e1-b7cc-1aacc3ce662e/5cf08dfe-d906-4adb-8c99-60cc69db1b65"
+          (reference "R15") (unit 1)
         )
       )
@@
     )
   )
+  (symbol (lib_id "Device:R_Small") (at 130.81 144.78 180) (unit 1)
+    (in_bom yes) (on_board yes) (dnp no) (fields_autoplaced)
+    (property "Reference" "R1" (at 133.35 143.51 0)
+      (effects (font (size 1.27 1.27)) (justify right))
+    )
+    (property "Value" "100k" (at 133.35 146.05 0)
+      (effects (font (size 1.27 1.27)) (justify right))
+    )
+    (property "Footprint" "passive:R_0402" (at 130.81 144.78 0)
+      (effects (font (size 1.27 1.27)) hide)
+    )
+    (property "Datasheet" "~" (at 130.81 144.78 0)
+      (effects (font (size 1.27 1.27)) hide)
+    )
+    (property "MFPN" "" (at 130.81 144.78 0)
+      (effects (font (size 1.27 1.27)) hide)
+    )
+    (property "Specification" "" (at 130.81 144.78 0)
+      (effects (font (size 1.27 1.27)) hide)
+    )
+    (pin "1")
+    (pin "2")
+    (instances
+      (project "battery-emulator"
+        (path "/7161d457-3f04-48e1-b7cc-1aacc3ce662e"
+          (reference "R1") (unit 1)
+        )
+        (path "/7161d457-3f04-48e1-b7cc-1aacc3ce662e/5cf08dfe-d906-4adb-8c99-60cc69db1b65"
+          (reference "R16") (unit 1)
+        )
+      )
+    )
+  )
   (symbol (lib_id "Device:C_Small") (at 196.85 109.22 0) (unit 1)
     (in_bom yes) (on_board yes) (dnp no) (fields_autoplaced)
@@
     )
   )
+  (symbol (lib_id "Device:C_Small") (at 140.97 144.78 0) (unit 1)
+    (in_bom yes) (on_board yes) (dnp no) (fields_autoplaced)
+    (property "Reference" "C3" (at 143.51 143.5163 0)
+      (effects (font (size 1.27 1.27)) (justify left))
+    )
+    (property "Value" "0.1u" (at 143.51 146.0563 0)
+      (effects (font (size 1.27 1.27)) (justify left))
+    )
+    (property "Footprint" "passive:C_0402" (at 140.97 144.78 0)
+      (effects (font (size 1.27 1.27)) hide)
+    )
+    (property "Datasheet" "~" (at 140.97 144.78 0)
+      (effects (font (size 1.27 1.27)) hide)
+    )
+    (property "MFPN" "" (at 140.97 144.78 0)
+      (effects (font (size 1.27 1.27)) hide)
+    )
+    (property "Specification" "" (at 140.97 144.78 0)
+      (effects (font (size 1.27 1.27)) hide)
+    )
+    (pin "1")
+    (pin "2")
+    (instances
+      (project "battery-emulator"
+        (path "/7161d457-3f04-48e1-b7cc-1aacc3ce662e"
+          (reference "C3") (unit 1)
+        )
+        (path "/7161d457-3f04-48e1-b7cc-1aacc3ce662e/5cf08dfe-d906-4adb-8c99-60cc69db1b65"
+          (reference "C25") (unit 1)
+        )
+      )
+    )
+  )
   (symbol (lib_id "Device:C_Small") (at 212.09 96.52 0) (unit 1)
     (in_bom yes) (on_board yes) (dnp no) (fields_autoplaced)
@@
         (path "/7161d457-3f04-48e1-b7cc-1aacc3ce662e/5cf08dfe-d906-4adb-8c99-60cc69db1b65"
           (reference "C1") (unit 1)
+        )
+      )
+    )
+  )
+  (symbol (lib_id "power:GND") (at 130.81 147.32 0) (unit 1)
+    (in_bom yes) (on_board yes) (dnp no) (fields_autoplaced)
+    (property "Reference" "#PWR011" (at 130.81 153.67 0)
+      (effects (font (size 1.27 1.27)) hide)
+    )
+    (property "Value" "GND" (at 130.81 151.13 90)
+      (effects (font (size 1.27 1.27)) (justify right) hide)
+    )
+    (property "Footprint" "" (at 130.81 147.32 0)
+      (effects (font (size 1.27 1.27)) hide)
+    )
+    (property "Datasheet" "" (at 130.81 147.32 0)
+      (effects (font (size 1.27 1.27)) hide)
+    )
+    (pin "1")
+    (instances
+      (project "battery-emulator"
+        (path "/7161d457-3f04-48e1-b7cc-1aacc3ce662e"
+          (reference "#PWR011") (unit 1)
+        )
+        (path "/7161d457-3f04-48e1-b7cc-1aacc3ce662e/5cf08dfe-d906-4adb-8c99-60cc69db1b65"
+          (reference "#PWR067") (unit 1)
         )
       )
@@
         )
       )
+    )
+  )
+  (symbol (lib_id "power:GND") (at 140.97 147.32 0) (unit 1)
+    (in_bom yes) (on_board yes) (dnp no) (fields_autoplaced)
+    (property "Reference" "#PWR011" (at 140.97 153.67 0)
+      (effects (font (size 1.27 1.27)) hide)
+    )
+    (property "Value" "GND" (at 140.97 151.13 90)
+      (effects (font (size 1.27 1.27)) (justify right) hide)
+    )
+    (property "Footprint" "" (at 140.97 147.32 0)
+      (effects (font (size 1.27 1.27)) hide)
+    )
+    (property "Datasheet" "" (at 140.97 147.32 0)
+      (effects (font (size 1.27 1.27)) hide)
+    )
+    (pin "1")
+    (instances
+      (project "battery-emulator"
+        (path "/7161d457-3f04-48e1-b7cc-1aacc3ce662e"
+          (reference "#PWR011") (unit 1)
+        )
+        (path "/7161d457-3f04-48e1-b7cc-1aacc3ce662e/5cf08dfe-d906-4adb-8c99-60cc69db1b65"
+          (reference "#PWR068") (unit 1)
+        )
+      )

Commit message: Layout complete
Parts:
- removed FB1: BLM18KG471SN1D, passive:R_0603, symbol Device:FerriteBead_Small
Connections:
- net V_{O,PROT} is gone; now on net OUTPUT: C2.1, C2.1, C2.1, D1.2 (A), D2.1 (K), R3.2, U2.5 (-)
- net +3.3V: now also C3.1, U2.3 (V+)
- net +5V: no longer C3.1, U2.3 (V+)
Changed lines of the file:
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@@
     (stroke (width 0) (type default))
   )
-  (wire (pts (xy 234.95 90.17) (xy 240.03 90.17))
+  (wire (pts (xy 222.25 90.17) (xy 234.95 90.17))
     (stroke (width 0) (type default))
   )
@@
   )
   (wire (pts (xy 123.19 139.7) (xy 130.81 139.7))
-    (stroke (width 0) (type default))
-  )
-  (wire (pts (xy 222.25 90.17) (xy 229.87 90.17))
     (stroke (width 0) (type default))
   )
@@
     (effects (font (size 1.27 1.27)) (justify left))
   )
-  (hierarchical_label "OUTPUT" (shape input) (at 240.03 90.17 0) (fields_autoplaced)
+  (hierarchical_label "OUTPUT" (shape input) (at 234.95 90.17 0) (fields_autoplaced)
     (effects (font (size 1.27 1.27)) (justify left))
   )
@@
   (hierarchical_label "I_{MEAS}" (shape input) (at 153.67 119.38 180) (fields_autoplaced)
     (effects (font (size 1.27 1.27)) (justify right))
-  )
-  (symbol (lib_id "Device:FerriteBead_Small") (at 232.41 90.17 90) (unit 1)
-    (in_bom yes) (on_board yes) (dnp no) (fields_autoplaced)
-    (property "Reference" "FB1" (at 232.3719 83.82 90)
-      (effects (font (size 1.27 1.27)))
-    )
-    (property "Value" "BLM18KG471SN1D" (at 232.3719 86.36 90)
-      (effects (font (size 1.27 1.27)))
-    )
-    (property "Footprint" "passive:R_0603" (at 232.41 91.948 90)
-      (effects (font (size 1.27 1.27)) hide)
-    )
-    (property "Datasheet" "~" (at 232.41 90.17 0)
-      (effects (font (size 1.27 1.27)) hide)
-    )
-    (pin "1")
-    (pin "2")
-    (instances
-      (project "battery-emulator"
-        (path "/7161d457-3f04-48e1-b7cc-1aacc3ce662e"
-          (reference "FB1") (unit 1)
-        )
-        (path "/7161d457-3f04-48e1-b7cc-1aacc3ce662e/5cf08dfe-d906-4adb-8c99-60cc69db1b65"
-          (reference "FB1") (unit 1)
-        )
-      )
-    )
   )
   (symbol (lib_id "power:GND") (at 71.12 106.68 0) (unit 1)
@@
     )
   )
-  (symbol (lib_id "power:+5V") (at 157.48 99.06 90) (unit 1)
-    (in_bom yes) (on_board yes) (dnp no) (fields_autoplaced)
-    (property "Reference" "#PWR07" (at 161.29 99.06 0)
-      (effects (font (size 1.27 1.27)) hide)
-    )
-    (property "Value" "+5V" (at 153.67 99.06 90)
-      (effects (font (size 1.27 1.27)) (justify left))
-    )
-    (property "Footprint" "" (at 157.48 99.06 0)
-      (effects (font (size 1.27 1.27)) hide)
-    )
-    (property "Datasheet" "" (at 157.48 99.06 0)
-      (effects (font (size 1.27 1.27)) hide)
-    )
-    (pin "1")
-    (instances
-      (project "battery-emulator"
-        (path "/7161d457-3f04-48e1-b7cc-1aacc3ce662e"
-          (reference "#PWR07") (unit 1)
-        )
-        (path "/7161d457-3f04-48e1-b7cc-1aacc3ce662e/5cf08dfe-d906-4adb-8c99-60cc69db1b65"
-          (reference "#PWR06") (unit 1)
-        )
-      )
-    )
-  )
   (symbol (lib_id "power:GND") (at 91.44 105.41 270) (unit 1)
     (in_bom yes) (on_board yes) (dnp no) (fields_autoplaced)
@@
         )
       )
+    )
+  )
+  (symbol (lib_id "power:+3.3V") (at 157.48 99.06 90) (unit 1)
+    (in_bom yes) (on_board yes) (dnp no) (fields_autoplaced)
+    (property "Reference" "#PWR09" (at 161.29 99.06 0)
+      (effects (font (size 1.27 1.27)) hide)
+    )
+    (property "Value" "+3.3V" (at 153.67 99.06 90)
+      (effects (font (size 1.27 1.27)) (justify left))
+    )
+    (property "Footprint" "" (at 157.48 99.06 0)
+      (effects (font (size 1.27 1.27)) hide)
+    )
+    (property "Datasheet" "" (at 157.48 99.06 0)
+      (effects (font (size 1.27 1.27)) hide)
+    )
+    (pin "1")
+    (instances
+      (project "rs-probe"
+        (path "/224768bc-6009-43ba-aa4a-70cbaa15b5a3"
+          (reference "#PWR09") (unit 1)
+        )
+      )
+      (project "battery-emulator"
+        (path "/7161d457-3f04-48e1-b7cc-1aacc3ce662e"
+          (reference "#PWR035") (unit 1)
+        )
+        (path "/7161d457-3f04-48e1-b7cc-1aacc3ce662e/5cf08dfe-d906-4adb-8c99-60cc69db1b65"
+          (reference "#PWR069") (unit 1)
+        )
+      )
