File: battery-emulator.kicad_pcb (KiCad board)
At the start: 4 copper layers, 40 x 40 mm, 52 parts, among them J1 USB_C_Receptacle_USB2.0, J2 tag-connect-swd, J3 FakeBattery, SW1 SW_Push, U1 OPA567AIRHGR, U2 INA199A1DCKR, U3 NUF2042XV6T1G, U4 W25Q8, U5 RP2040, U6 NCP161ASN330T1G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

Commit message: More layout
Parts:
- added C25: 0.1u, passive:C_0402, F.Cu at (110.8, 124.8)
- added R15: 100k, passive:R_0402, F.Cu at (109.4, 125.3)
- added R16: 100k, passive:R_0402, F.Cu at (109.4, 124.3)
- added SW2: SW_Push, Button_Switch_SMD:SW_SPST_EVQP2, F.Cu at (125.0, 110.0)
- added SW3: SW_Push, Button_Switch_SMD:SW_SPST_EVQP2, F.Cu at (125.0, 130.0)
- added SW4: SW_Push, Button_Switch_SMD:SW_SPST_EVQP2, F.Cu at (125.0, 120.0)
- moved U4 70.4 mm to (110.0, 117.3), turned to 90 degrees
- moved R7 61.9 mm to (107.7, 118.6), turned to 180 degrees
- moved U5 61.3 mm to (115.5, 115.0), turned to 90 degrees
- moved C5 59.4 mm to (108.2, 116.4), turned to -90 degrees
- moved U3 58.9 mm to (110.0, 108.9), turned to 90 degrees
- moved J1 47.9 mm to (110.5, 102.5), turned to 180 degrees
- moved U6 26.9 mm to (142.1, 83.5)
- moved C1 2.50 mm to (110.7, 122.8)
- moved C17 2.50 mm to (107.0, 129.5)
- moved C2 2.50 mm to (113.7, 122.9)
- moved C20 2.50 mm to (118.8, 124.0)
- moved C21 2.50 mm to (118.8, 126.0)
- moved C22 2.50 mm to (105.2, 127.6)
- moved C23 2.50 mm to (103.8, 124.5)
- moved C24 2.50 mm to (101.3, 124.5)
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Connections:
- U5 pad 12: /TEMP0 -> unconnected-(U5-GPIO9-Pad12)
- U5 pad 13: /CURR0 -> unconnected-(U5-GPIO10-Pad13)
- U5 pad 14: /ENABLE0 -> unconnected-(U5-GPIO11-Pad14)
- U5 pad 3: unconnected-(U5-GPIO1-Pad3) -> /TEMP0
- U5 pad 39: unconnected-(U5-GPIO27_ADC1-Pad39) -> /VMEAS_0
- U5 pad 4: /VREF_1 -> /CURR0
- U5 pad 5: unconnected-(U5-GPIO3-Pad5) -> /ENABLE0
- U5 pad 6: /VREF_2 -> unconnected-(U5-GPIO4-Pad6)
- U5 pad 7: unconnected-(U5-GPIO5-Pad7) -> /SW1
- U5 pad 8: /VREF_3 -> /SW2
- U5 pad 9: unconnected-(U5-GPIO7-Pad9) -> /SW3
Routing:
- net /Power stage/V_{O}: track 1.78 -> 17.4 mm
- net +5V: track 8.51 -> 16.5 mm, vias 3 -> 10
- net Net-(U4-~{CS}): track 0.00 -> 4.68 mm
- net Net-(U4-DO(IO1)): track 0.00 -> 4.23 mm
- net GND: track 2.81 -> 6.29 mm, vias 19 -> 59
- net Net-(U4-IO2): track 0.00 -> 3.15 mm
- net Net-(U4-IO3): track 0.00 -> 3.00 mm
- net Net-(U4-CLK): track 0.00 -> 2.54 mm
- net /VMEAS_0: track 0.00 -> 1.97 mm
- net /D_P: track 0.00 -> 1.76 mm
- net /D_N: track 0.00 -> 1.76 mm
- net +3.3V: track 0.00 -> 1.68 mm, vias 0 -> 1
- net Net-(U4-DI(IO0)): track 0.00 -> 1.63 mm
- net Net-(U1-I_{SET}): track 3.32 -> 2.65 mm
- net /CURR0: track 2.79 -> 2.94 mm, vias 0 -> 1
Other:
- outline, holes or cut-outs redrawn

Commit message: Layout complete
Parts:
- added FB2: BLM18KG471SN1D, passive:R_0603, F.Cu at (101.3, 127.4)
- moved SW1 69.4 mm to (104.5, 115.4), turned to 90 degrees
- moved R5 59.6 mm to (104.7, 105.6), turned to -90 degrees
- moved C8 53.8 mm to (109.0, 114.0), turned to 180 degrees
- moved C6 53.5 mm to (110.3, 111.6), turned to 180 degrees
- moved R6 53.4 mm to (121.0, 119.3)
- moved C7 53.0 mm to (110.3, 112.6), turned to 180 degrees
- moved C13 53.0 mm to (112.5, 110.1), turned to 180 degrees
- moved C10 52.5 mm to (112.4, 120.0), turned to 180 degrees
- moved C16 51.6 mm to (117.9, 120.0)
- moved C11 51.2 mm to (109.0, 114.9), turned to 180 degrees
- moved C12 50.6 mm to (117.0, 110.1)
- moved R4 50.5 mm to (116.3, 105.6), turned to -90 degrees
- moved X1 50.0 mm to (121.0, 117.3), turned to 90 degrees
- moved J2 48.4 mm to (126.4, 115.0)
- moved C15 47.3 mm to (121.0, 115.2)
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Connections:
- net /Power stage/OUTPUT renamed Net-(J3-Pin_1)
- net Net-(U5-XIN) renamed /XIN
- C3 pad 1: +5V -> +3.3V
- J3 pad 2: GND -> Net-(J3-Pin_2)
- U2 pad 3: +5V -> +3.3V
- U5 pad 14: unconnected-(U5-GPIO11-Pad14) -> /SW2
- U5 pad 15: unconnected-(U5-GPIO12-Pad15) -> /SW3
- U5 pad 28: unconnected-(U5-GPIO17-Pad28) -> /SW1
- U5 pad 3: /TEMP0 -> /ENABLE0
- U5 pad 4: /CURR0 -> /TEMP0
- U5 pad 5: /ENABLE0 -> /CURR0
- U5 pad 7: /SW1 -> unconnected-(U5-GPIO5-Pad7)
- U5 pad 8: /SW2 -> unconnected-(U5-GPIO6-Pad8)
- U5 pad 9: /SW3 -> unconnected-(U5-GPIO7-Pad9)
Routing:
- net +3.3V: track 1.68 -> 92.9 mm, vias 1 -> 14
- net /VMEAS_0: track 1.97 -> 41.4 mm, vias 0 -> 2
- net /IMEAS_0: track 0.97 -> 39.5 mm, vias 0 -> 2
- net +1V1: track 0.00 -> 18.4 mm, vias 0 -> 3
- net /SW2: track 0.00 -> 18.1 mm
- net /CURR0: track 2.94 -> 17.2 mm, vias 1 -> 2
- net /SW3: track 0.00 -> 12.0 mm
- net /SW1: track 0.00 -> 10.3 mm
- net GND: track 6.29 -> 14.9 mm, vias 59 -> 464
- net /P_SWCLK: track 0.00 -> 7.95 mm
- net /VREF_0: track 0.00 -> 7.75 mm
- net /D_FS_P: track 0.00 -> 7.62 mm
- net /P_SWDIO: track 0.00 -> 7.46 mm, vias 0 -> 2
- net Net-(R7-Pad2): track 0.00 -> 7.26 mm
- net /D_FS_N: track 0.00 -> 7.26 mm
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- added copper zone on In2.Cu, net +5V
Other:
- board text added: "+"
- board text added: "-"
- board text added: "BATTERY OUT 1.5A MAX"
- board text added: "EMPTY"
- board text added: "FULL"
- board text added: "HALF"
- board text added: "LiPo Emulator"

Commit message: More fixes
Parts:
- added FB3: BLM18KG471SN1D, passive:R_0603, F.Cu at (114.3, 108.5)
Connections:
- C18 pad 1: +5V -> Net-(U6-EN)
- U6 pad 1: +5V -> Net-(U6-EN)
- U6 pad 3: +5V -> Net-(U6-EN)
Routing:
- net GND: track 14.9 -> 23.4 mm, vias 464 -> 494
- net +5V: track 23.1 -> 15.8 mm
- net Net-(U6-EN): track 0.00 -> 6.46 mm
Other:
- board text added: "Battery Emulator"
- board text removed: "LiPo Emulator"
