File: battery-emulator.kicad_sch (KiCad schematic)
At the start: 11 parts, among them U1 INA199A1DCKR

Commit message: Some design
Parts:
- removed C2: 47u, passive:C_1206, symbol Device:C_Small
- removed C4: 330u, Capacitor_SMD:C_Elec_8x10.2, symbol Device:C_Polarized_Small
- removed D1, D2: 1A, 40V, Diode_SMD:D_SOD-323, symbol Device:D_Schottky_Small
- removed R1: 10k, symbol Device:R_Small
- removed U1: INA199A1DCKR, Package_TO_SOT_SMD:SOT-363_SC-70-6, symbol Amplifier_Current:INA199xxDCK
- removed U?: OPA567AIRHGR, qfn:PVQFN-N12-1EP_5.0x5.0mm_P1.0mm_EP3.12x3.12mm, symbol opamp:OPA567
- added C10, C11, C12, C13, C14, C18, C7, C9: 0.1u, passive:C_0402, symbol Device:C_Small
- added C4 (x3), C6: 2.2u, passive:C_0402, symbol Device:C_Small
- added J1: USB_C_Receptacle_USB2.0, connectors:USB_C_Receptacle_USB4105, symbol Connector:USB_C_Receptacle_USB2.0
- added J3: FakeBattery, Connector_JST:JST_PH_S2B-PH-SM4-TB_1x02-1MP_P2.00mm_Horizontal, symbol Connector_Generic_MountingPin:Conn_01x02_MountingPin
- added J5: tag-connect-swd, Connector:Tag-Connect_TC2030-IDC-NL_2x03_P1.27mm_Vertical, symbol connectors:tag-connect-swd
- added R17: 1k, passive:R_0402, symbol Device:R_Small
- added R4: 5.1k, passive:R_0402, symbol Device:R_Small
- added SW1: SW_Push, Button_Switch_SMD:SW_SPST_EVQP2, symbol Switch:SW_Push
- added U3: W25Q8, son:USON-8-3x2mm-EP, symbol Memory_Flash:W25Q32JVZP
- added U6: RP2040, qfn:RP2040-QFN-56, symbol rp2040:RP2040
- added U6: NCP161ASN330T1G, sot:SOT-23-5, symbol ldo:NCP161ASN300T1G
- added U7: NUF2042XV6T1G, sot:SOT-563, symbol interface_esd:NUF2042XV6T1G
- added X1: 12 MHz, crystals:Crystal_SMD_2520-4Pin_2.5x2.0mm, symbol Oscillator:ASCO
- C1: LCSC (none) -> C56392; Tolerance (none) -> 25V, X7R
- C3: value 0.1u -> 2.2u; LCSC (none) -> C77002; Tolerance (none) -> 10V, X5R
- R2: value 10k -> 1k; footprint (none) -> passive:R_0402; LCSC (none) -> C106235; Tolerance (none) -> 1%
- R3: value 20m -> 5.1k; footprint (none) -> passive:R_0402; LCSC (none) -> C105872; Tolerance (none) -> 1%
Connections:
- net +5V: now also C4.1, J1.A4 (VBUS), J1.A9 (VBUS), J1.B4 (VBUS), J1.B9 (VBUS), U6.1 (VIN), U6.3 (EN), U7.5 (VBUS); no longer C1.1, C3.1
- net GND: now also R3.2, C10.2, C11.2, C12.2, C13.2, C14.2, C18.2, C4.2, C4.2, C4.2, C6.2, C7.2, C9.2, J1.A1 (GND), J1.A12 (GND), J1.B1 (GND), J1.B12 (GND), J1.S1 (SHIELD), J3.2 (Pin_2), J3.MP (MountPin), J5.5 (GND), R4.2, SW1.1, U3.4 (GND), U3.9 (EP), U6.19 (TESTEN), U6.2 (GND), U6.57 (GND), U7.2 (GND), X1.2 (GND); no longer R2.1
- net at R3.1: now also J1.A5 (CC1)
- net at R2.2: now also SW1.2
- new net: J1.B5 (CC2), R4.1
- new net: R17.2, X1.1 (Tri-State)
- new net: R2.1, U3.1 (~{CS}), U6.56 (QSPI_SS)
- new net: U6.20 (XIN), X1.3 (OUT)
- new net: U3.7 (IO3), U6.51 (QSPI_SD3)
- new net: U3.6 (CLK), U6.52 (QSPI_SCLK)
- new net: U3.5 (DI(IO0)), U6.53 (QSPI_SD0)
- new net: U3.3 (IO2), U6.54 (QSPI_SD2)
- new net: U3.2 (DO(IO1)), U6.55 (QSPI_SD1)
- new net +1V1: C10.1, C4.1, C7.1, U6.23 (DVDD), U6.45 (VREG_VOUT), U6.50 (DVDD)
- new net +3.3V: C1.1, C11.1, C12.1, C13.1, C14.1, C18.1, C3.1, C4.1, C6.1, C9.1, J5.1 (VCC), R17.1, U3.8 (VCC), U6.1 (IOVDD), U6.10 (IOVDD), U6.22 (IOVDD), U6.26 (RUN), U6.33 (IOVDD), U6.42 (IOVDD), U6.43 (ADC_AVDD), U6.44 (VREG_IN), U6.48 (USB_VDD), U6.49 (IOVDD), U6.5 (VOUT), X1.4 (VDD)
- new net CURR0: U6.13 (GPIO10)
- new net D_FS_N: U6.46 (USB_DM), U7.3 (D2I)
- new net D_FS_P: U6.47 (USB_DP), U7.1 (D1I)
- new net D_N: J1.A7 (D-), J1.B7 (D-), U7.4 (D2O)
- new net D_P: J1.A6 (D+), J1.B6 (D+), U7.6 (D1O)
- new net ENABLE0: U6.14 (GPIO11)
- new net IMEAS_0: U6.38 (GPIO26_ADC0)
- new net P_SWCLK: J5.4 (SWCLK), U6.24 (SWCLK)
- new net P_SWDIO: J5.2 (SWDIO), U6.25 (SWD)
- new net Power stage/OUTPUT: J3.1 (Pin_1)
- new net TEMP0: U6.12 (GPIO9)
- new net VREF_0: U6.2 (GPIO0)
- new net VREF_1: U6.4 (GPIO2)
- new net VREF_2: U6.6 (GPIO4)
- new net VREF_3: U6.8 (GPIO6)
- no-connect marks 0 -> 5
Other:
- added sheet Power stage (power_stage.kicad_sch)
- note added: "DESIGN NOTE: Hold button during power up to enter USB bootloader."
- note removed: "DESIGN NOTE: Gain = 2"
- note removed: "DESIGN NOTE: Gain = 50"

Commit message: More layout
Parts:
- added SW1 (x3): SW_Push, Button_Switch_SMD:SW_SPST_EVQP2, symbol Switch:SW_Push
Connections:
- net VREF_1 is gone; now on net CURR0: U6.4 (GPIO2)
- net CURR0: no longer U6.13 (GPIO10)
- net ENABLE0: now also U6.5 (GPIO3); no longer U6.14 (GPIO11)
- net GND: now also SW1.1, SW1.1, SW1.1
- net TEMP0: now also U6.3 (GPIO1); no longer U6.12 (GPIO9)
- net VMEAS_0: now reaches U6.39 (GPIO27_ADC1)
- net SW1: now reaches U6.7 (GPIO5)
- net SW1: now also SW1.2
- net SW3: now reaches U6.9 (GPIO7)
- net SW3: now also SW1.2
- net VREF_2: no longer names the net of U6.6 (GPIO4)
- net VREF_3 renamed SW2
- net SW2: now also SW1.2
Other:
- sheet Power stage ports: added V_{MEAS}; removed none

Commit message: Layout complete
Parts:
- added FB1, FB2: BLM18KG471SN1D, passive:R_0603, symbol Device:FerriteBead_Small
Connections:
- net CURR0: now also U6.5 (GPIO3); no longer U6.4 (GPIO2)
- net ENABLE0: now also U6.3 (GPIO1); no longer U6.5 (GPIO3)
- net GND: now also FB2.1; no longer J3.2 (Pin_2)
- net Power stage/OUTPUT: now also FB1.1; no longer J3.1 (Pin_1)
- net SW1: now also U6.28 (GPIO17); no longer U6.7 (GPIO5)
- net SW2: now also U6.14 (GPIO11); no longer U6.8 (GPIO6)
- net SW3: now also U6.15 (GPIO12); no longer U6.9 (GPIO7)
- net TEMP0: now also U6.4 (GPIO2); no longer U6.3 (GPIO1)
- net XIN: now reaches U6.20 (XIN), X1.3 (OUT)
- new net: FB1.2, J3.1 (Pin_1)
- new net: FB2.2, J3.2 (Pin_2)
Other:
- moved on the sheet: J3
Changed lines of the file:
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@@
     (stroke (width 0) (type default))
   )
-  (wire (pts (xy 222.25 40.64) (xy 238.76 40.64))
+  (wire (pts (xy 222.25 40.64) (xy 231.14 40.64))
     (stroke (width 0) (type default))
   )
@@
     (stroke (width 0) (type default))
   )
+  (wire (pts (xy 251.46 43.18) (xy 247.65 43.18))
+    (stroke (width 0) (type default))
+  )
   (wire (pts (xy 54.61 49.53) (xy 63.5 49.53))
     (stroke (width 0) (type default))
@@
     (stroke (width 0) (type default))
   )
+  (wire (pts (xy 247.65 43.18) (xy 247.65 45.72))
+    (stroke (width 0) (type default))
+  )
   (wire (pts (xy 81.28 35.56) (xy 90.17 35.56))
     (stroke (width 0) (type default))
@@
   )
   (wire (pts (xy 233.68 134.62) (xy 233.68 135.89))
+    (stroke (width 0) (type default))
+  )
+  (wire (pts (xy 236.22 40.64) (xy 251.46 40.64))
     (stroke (width 0) (type default))
   )
@@
     (effects (font (size 1.27 1.27)) (justify left bottom))
   )
-  (label "SW1" (at 128.27 105.41 0) (fields_autoplaced)
+  (label "SW1" (at 128.27 135.89 0) (fields_autoplaced)
     (effects (font (size 1.27 1.27)) (justify left bottom))
   )
-  (label "CURR0" (at 128.27 97.79 0) (fields_autoplaced)
+  (label "CURR0" (at 128.27 100.33 0) (fields_autoplaced)
     (effects (font (size 1.27 1.27)) (justify left bottom))
   )
@@
     (effects (font (size 1.27 1.27)) (justify right bottom))
   )
+  (label "XIN" (at 64.77 128.27 180) (fields_autoplaced)
+    (effects (font (size 1.27 1.27)) (justify right bottom))
+  )
   (label "D_FS_N" (at 201.93 130.81 180) (fields_autoplaced)
     (effects (font (size 1.27 1.27)) (justify right bottom))
@@
     (effects (font (size 1.27 1.27)) (justify right bottom))
   )
-  (label "SW2" (at 128.27 107.95 0) (fields_autoplaced)
+  (label "SW2" (at 128.27 120.65 0) (fields_autoplaced)
     (effects (font (size 1.27 1.27)) (justify left bottom))
   )
-  (label "ENABLE0" (at 128.27 100.33 0) (fields_autoplaced)
+  (label "ENABLE0" (at 128.27 95.25 0) (fields_autoplaced)
     (effects (font (size 1.27 1.27)) (justify left bottom))
   )
@@
     (effects (font (size 1.27 1.27)) (justify left bottom))
   )
-  (label "SW3" (at 128.27 110.49 0) (fields_autoplaced)
+  (label "SW3" (at 128.27 123.19 0) (fields_autoplaced)
     (effects (font (size 1.27 1.27)) (justify left bottom))
   )
@@
     (effects (font (size 1.27 1.27)) (justify right bottom))
   )
-  (label "TEMP0" (at 128.27 95.25 0) (fields_autoplaced)
+  (label "TEMP0" (at 128.27 97.79 0) (fields_autoplaced)
     (effects (font (size 1.27 1.27)) (justify left bottom))
   )
@@
     )
   )
-  (symbol (lib_id "power:GND") (at 243.84 48.26 0) (unit 1)
-    (in_bom yes) (on_board yes) (dnp no)
-    (property "Reference" "#PWR012" (at 243.84 54.61 0)
-      (effects (font (size 1.27 1.27)) hide)
-    )
-    (property "Value" "GND" (at 243.967 52.6542 0)
-      (effects (font (size 1.27 1.27)) hide)
-    )
-    (property "Footprint" "" (at 243.84 48.26 0)
-      (effects (font (size 1.27 1.27)) hide)
-    )
-    (property "Datasheet" "" (at 243.84 48.26 0)
+  (symbol (lib_id "power:GND") (at 256.54 48.26 0) (unit 1)
+    (in_bom yes) (on_board yes) (dnp no)
+    (property "Reference" "#PWR012" (at 256.54 54.61 0)
+      (effects (font (size 1.27 1.27)) hide)
+    )
+    (property "Value" "GND" (at 256.667 52.6542 0)
+      (effects (font (size 1.27 1.27)) hide)
+    )
+    (property "Footprint" "" (at 256.54 48.26 0)
+      (effects (font (size 1.27 1.27)) hide)
+    )
+    (property "Datasheet" "" (at 256.54 48.26 0)
       (effects (font (size 1.27 1.27)) hide)
     )
@@
         (path "/7161d457-3f04-48e1-b7cc-1aacc3ce662e"
           (reference "#PWR061") (unit 1)
+        )
+      )
+    )
+  )
+  (symbol (lib_id "Device:FerriteBead_Small") (at 233.68 40.64 90) (unit 1)
+    (in_bom yes) (on_board yes) (dnp no) (fields_autoplaced)
+    (property "Reference" "FB1" (at 233.6419 34.29 90)
+      (effects (font (size 1.27 1.27)))
+    )
+    (property "Value" "BLM18KG471SN1D" (at 233.6419 36.83 90)
+      (effects (font (size 1.27 1.27)))
+    )
+    (property "Footprint" "passive:R_0603" (at 233.68 42.418 90)
+      (effects (font (size 1.27 1.27)) hide)
+    )
+    (property "Datasheet" "~" (at 233.68 40.64 0)
+      (effects (font (size 1.27 1.27)) hide)
+    )
+    (pin "1")
+    (pin "2")
+    (instances
+      (project "battery-emulator"
+        (path "/7161d457-3f04-48e1-b7cc-1aacc3ce662e"
+          (reference "FB1") (unit 1)
+        )
+        (path "/7161d457-3f04-48e1-b7cc-1aacc3ce662e/5cf08dfe-d906-4adb-8c99-60cc69db1b65"
+          (reference "FB1") (unit 1)
         )
       )
@@
         (path "/7161d457-3f04-48e1-b7cc-1aacc3ce662e"
           (reference "#PWR014") (unit 1)
+        )
+      )
+    )
+  )
+  (symbol (lib_id "Device:FerriteBead_Small") (at 247.65 48.26 180) (unit 1)
+    (in_bom yes) (on_board yes) (dnp no) (fields_autoplaced)
+    (property "Reference" "FB2" (at 245.11 47.0281 0)
+      (effects (font (size 1.27 1.27)) (justify left))
+    )
+    (property "Value" "BLM18KG471SN1D" (at 245.11 49.5681 0)
+      (effects (font (size 1.27 1.27)) (justify left))
+    )
+    (property "Footprint" "passive:R_0603" (at 249.428 48.26 90)
+      (effects (font (size 1.27 1.27)) hide)
+    )
+    (property "Datasheet" "~" (at 247.65 48.26 0)
+      (effects (font (size 1.27 1.27)) hide)
+    )
+    (pin "1")
+    (pin "2")
+    (instances
+      (project "battery-emulator"
+        (path "/7161d457-3f04-48e1-b7cc-1aacc3ce662e"
+          (reference "FB2") (unit 1)
+        )
+        (path "/7161d457-3f04-48e1-b7cc-1aacc3ce662e/5cf08dfe-d906-4adb-8c99-60cc69db1b65"
+          (reference "FB1") (unit 1)
         )
       )
@@
     )
   )
-  (symbol (lib_id "Connector_Generic_MountingPin:Conn_01x02_MountingPin") (at 243.84 40.64 0) (unit 1)
+  (symbol (lib_id "Connector_Generic_MountingPin:Conn_01x02_MountingPin") (at 256.54 40.64 0) (unit 1)
     (in_bom yes) (on_board yes) (dnp no) (fields_autoplaced)
-    (property "Reference" "J3" (at 246.38 40.64 0)
-      (effects (font (size 1.27 1.27)) (justify left))
-    )
-    (property "Value" "FakeBattery" (at 246.38 43.18 0)
-      (effects (font (size 1.27 1.27)) (justify left))
-    )
-    (property "Footprint" "Connector_JST:JST_PH_S2B-PH-SM4-TB_1x02-1MP_P2.00mm_Horizontal" (at 243.84 40.64 0)
-      (effects (font (size 1.27 1.27)) hide)
-    )
-    (property "Datasheet" "~" (at 243.84 40.64 0)
-      (effects (font (size 1.27 1.27)) hide)
-    )
-    (property "MFPN" "" (at 243.84 40.64 0)
-      (effects (font (size 1.27 1.27)) hide)
-    )
-    (property "Specification" "" (at 243.84 40.64 0)
+    (property "Reference" "J3" (at 259.08 40.64 0)
+      (effects (font (size 1.27 1.27)) (justify left))
+    )
+    (property "Value" "FakeBattery" (at 259.08 43.18 0)
+      (effects (font (size 1.27 1.27)) (justify left))
+    )
+    (property "Footprint" "Connector_JST:JST_PH_S2B-PH-SM4-TB_1x02-1MP_P2.00mm_Horizontal" (at 256.54 40.64 0)
+      (effects (font (size 1.27 1.27)) hide)
+    )
+    (property "Datasheet" "~" (at 256.54 40.64 0)
+      (effects (font (size 1.27 1.27)) hide)
+    )
+    (property "MFPN" "" (at 256.54 40.64 0)
+      (effects (font (size 1.27 1.27)) hide)
+    )
+    (property "Specification" "" (at 256.54 40.64 0)
       (effects (font (size 1.27 1.27)) hide)
     )
@@
     )
   )
-  (symbol (lib_id "power:GND") (at 238.76 43.18 0) (unit 1)
-    (in_bom yes) (on_board yes) (dnp no)
-    (property "Reference" "#PWR012" (at 238.76 49.53 0)
-      (effects (font (size 1.27 1.27)) hide)
-    )
-    (property "Value" "GND" (at 238.887 47.5742 0)
-      (effects (font (size 1.27 1.27)) hide)
-    )
-    (property "Footprint" "" (at 238.76 43.18 0)
-      (effects (font (size 1.27 1.27)) hide)
-    )
-    (property "Datasheet" "" (at 238.76 43.18 0)
-      (effects (font (size 1.27 1.27)) hide)
-    )
+  (symbol (lib_id "power:GND") (at 247.65 50.8 0) (unit 1)
+    (in_bom yes) (on_board yes) (dnp no)
+    (property "Reference" "#PWR012" (at 247.65 57.15 0)
+      (effects (font (size 1.27 1.27)) hide)
+    )
+    (property "Value" "GND" (at 247.777 55.1942 0)
+      (effects (font (size 1.27 1.27)) hide)
+    )
+    (property "Footprint" "" (at 247.65 50.8 0)
+      (effects (font (size 1.27 1.27)) hide)
+    )
+    (property "Datasheet" "" (at 247.65 50.8 0)
+      (effects (font (size 1.27 1.27)) hide)
+    )

Commit message: More fixes
Parts:
- added FB3: BLM18KG471SN1D, passive:R_0603, symbol Device:FerriteBead_Small
- C3, C4, C6: value 2.2u -> 4.7u
Connections:
- net +5V: now also FB3.1; no longer C4.1, U6.1 (VIN), U6.3 (EN)
- new net: C4.1, FB3.2, U6.1 (VIN), U6.3 (EN)
Changed lines of the file:
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@@
+    (stroke (width 0) (type default))
+  )
+  (wire (pts (xy 201.93 90.17) (xy 210.82 90.17))
     (stroke (width 0) (type default))
   )
@@
     )
   )
-  (symbol (lib_id "power:+5V") (at 215.9 90.17 90) (unit 1)
-    (in_bom yes) (on_board yes) (dnp no)
-    (property "Reference" "#PWR024" (at 219.71 90.17 0)
-      (effects (font (size 1.27 1.27)) hide)
-    )
-    (property "Value" "+5V" (at 211.5058 89.789 0)
-      (effects (font (size 1.27 1.27)))
-    )
-    (property "Footprint" "" (at 215.9 90.17 0)
-      (effects (font (size 1.27 1.27)) hide)
-    )
-    (property "Datasheet" "" (at 215.9 90.17 0)
+  (symbol (lib_id "power:+5V") (at 201.93 90.17 90) (unit 1)
+    (in_bom yes) (on_board yes) (dnp no)
+    (property "Reference" "#PWR024" (at 205.74 90.17 0)
+      (effects (font (size 1.27 1.27)) hide)
+    )
+    (property "Value" "+5V" (at 197.5358 89.789 0)
+      (effects (font (size 1.27 1.27)))
+    )
+    (property "Footprint" "" (at 201.93 90.17 0)
+      (effects (font (size 1.27 1.27)) hide)
+    )
+    (property "Datasheet" "" (at 201.93 90.17 0)
       (effects (font (size 1.27 1.27)) hide)
     )
@@
       (effects (font (size 1.27 1.27)) (justify left))
     )
-    (property "Value" "2.2u" (at 48.0568 54.483 0)
+    (property "Value" "4.7u" (at 48.0568 54.483 0)
       (effects (font (size 1.27 1.27)) (justify left))
     )
@@
       (effects (font (size 1.27 1.27)) (justify left))
     )
-    (property "Value" "2.2u" (at 257.6068 97.663 0)
+    (property "Value" "4.7u" (at 257.6068 97.663 0)
       (effects (font (size 1.27 1.27)) (justify left))
     )
@@
       (effects (font (size 1.27 1.27)) (justify left))
     )
-    (property "Value" "2.2u" (at 48.0568 40.513 0)
+    (property "Value" "4.7u" (at 48.0568 40.513 0)
       (effects (font (size 1.27 1.27)) (justify left))
     )
@@
       (effects (font (size 1.27 1.27)) (justify left))
     )
-    (property "Value" "2.2u" (at 222.0468 97.663 0)
+    (property "Value" "4.7u" (at 222.0468 97.663 0)
       (effects (font (size 1.27 1.27)) (justify left))
     )
@@
       (effects (font (size 1.27 1.27)) (justify left))
     )
-    (property "Value" "2.2u" (at 56.9468 40.513 0)
+    (property "Value" "4.7u" (at 56.9468 40.513 0)
       (effects (font (size 1.27 1.27)) (justify left))
     )
@@
         )
       )
+    )
+  )
+  (symbol (lib_id "Device:FerriteBead_Small") (at 213.36 90.17 90) (unit 1)
+    (in_bom yes) (on_board yes) (dnp no) (fields_autoplaced)
+    (property "Reference" "FB3" (at 213.3219 83.82 90)
+      (effects (font (size 1.27 1.27)))
+    )
+    (property "Value" "BLM18KG471SN1D" (at 213.3219 86.36 90)
+      (effects (font (size 1.27 1.27)))
+    )
+    (property "Footprint" "passive:R_0603" (at 213.36 91.948 90)
+      (effects (font (size 1.27 1.27)) hide)
+    )
+    (property "Datasheet" "~" (at 213.36 90.17 0)
+      (effects (font (size 1.27 1.27)) hide)
+    )
+    (pin "1")
+    (pin "2")
+    (instances
+      (project "battery-emulator"
+        (path "/7161d457-3f04-48e1-b7cc-1aacc3ce662e"
+          (reference "FB3") (unit 1)
+        )
+        (path "/7161d457-3f04-48e1-b7cc-1aacc3ce662e/5cf08dfe-d906-4adb-8c99-60cc69db1b65"
+          (reference "FB1") (unit 1)
+        )
+      )
